File: boards/board-l/board-l.kicad_sch (KiCad schematic)
At the start: 71 parts, among them J2 B6B-XH-A(LF)(SN), J3 SWD 1x5 (hand-fit), J4 UART pads, SW1 EC11 15-detent, U2 AL8860MP-13, U3 STM32G031F8P6, U4 AP63203WU-7

Commit message: NTC divider R26: 10k -> 100k (line-c25803), regen board-l
The as-built 10 kOhm divider drew 168 uA worst case at 25 C, 1.68x
Murata's 0.1 mA operating-current maximum (fact-c13564-max-current).
100 kOhm gives 33.6 uA worst case (2.97x margin, holds under a
shorted-thermistor fault); 33 kOhm was evaluated and rejected since its
NTC-shorted asymptote already exceeds the limit. Uses the existing
line-c25803 (already placed at board-p R11) instead of a new
inventory line, moving its footprint to R0603 to match board-p R11 and
satisfy validate.py's per-LCSC package-consistency check. No encoder
change: Alps manufacturer-primary retrieval failed (part-specific 403)
and mirror-only evidence cannot correct a GUARANTEED_ELECTRICAL claim.

Registry/generator sync per the locked Wave-4 spec (issue #48,
decisions recorded in circuit-recheck-decisions.md):
- board_l_spec.py: R26 tuple -> 0603WAF1003T5E/100k/C25803/R0603;
  regenerated board-l.kicad_sch (idempotent on a second run)
- inventory.json: move R26 placement from line-c17414 to line-c25803
  (32/29/3 totals unchanged)
- component-project-passives/interactions.json: note the new R26
  placement and the encoder pull-up reference no longer served by
  line-c17414's NTC role
- circuit-spec-integration/rules.json: rule-ntc-adc-firmware now cites
  rec-c25803/fact-c25803-*; rule-al8860-led-stage gains
  fact-c2934070-tolerance; both gain conditioned_calculations verified
  against validate.py's arithmetic() evaluator
- forward-tests.json: mcu-led-thermal-change direct_record_ids swapped
  to match the rule record_ids union
- component-murata-ncp18xh103f03rb/SKILL.md: fix "maximum measurement
  current" -> "maximum operating current" wording (the #44 finding);
  name R26's new value in the divider description
Parts:
- R26: value 10k -> 100k; footprint zudo-led-lamp:R0805 -> zudo-led-lamp:R0603; symbol zudo-led-lamp:0805W8F1002T5E -> zudo-led-lamp:0603WAF1003T5E; LCSC C17414 -> C25803
Changed lines of the file:
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@@
 	)
 	(symbol
-		(lib_id "zudo-led-lamp:0805W8F1002T5E")
+		(lib_id "zudo-led-lamp:0603WAF1003T5E")
 		(at 358.14 177.8 0)
 		(unit 1)
@@
 			)
 		)
-		(property "Value" "10k"
+		(property "Value" "100k"
 			(at 358.14 182.88 0)
 			(effects
@@
 			)
 		)
-		(property "Footprint" "zudo-led-lamp:R0805"
+		(property "Footprint" "zudo-led-lamp:R0603"
 			(at 358.14 177.8 0)
 			(effects
@@
 			)
 		)
-		(property "LCSC" "C17414"
+		(property "LCSC" "C25803"
 			(at 358.14 185.42 0)
 			(effects
