File: boards/board-l/board-l.kicad_sch (KiCad schematic)
At the start: 71 parts, among them J2 B6B-XH-A(LF)(SN), J3 SWD 1x5 (hand-fit), J4 UART pads, SW1 EC11 15-detent, U2 AL8860MP-13, U3 STM32G031F8P6, U4 AP63203WU-7

Commit message: fix(schgen): keep bare-copper pad groups out of the assembly BOM
next-steps.mdx requires footprint-only pad groups to be absent from the
assembly BOM, but in_bom was hardcoded yes and the DNP flags disagreed:
board-l J4 was dnp=True while board-p J2/J3 and board-l TP1 were False.
A JLCPCB import would have carried placement rows with blank part
numbers.

in_bom is now derived from the LCSC field — an orderable line always has
one, bare copper never does — and J4's misleading DNP marker is dropped.
The three real DNP lines (D6/D7, R17/R18, board-l J3) keep in_bom=yes,
dnp=yes since they are purchasable.

Co-Authored-By: Claude Opus 5 (1M context) <noreply@anthropic.com>
Parts:
- J4: now fitted; now left out of the parts list
- TP1: now left out of the parts list
Changed lines of the file:
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@@
 		(unit 1)
 		(exclude_from_sim no)
-		(in_bom yes)
-		(on_board yes)
-		(dnp yes)
+		(in_bom no)
+		(on_board yes)
+		(dnp no)
 		(property "Reference" "J4"
 			(at 241.3 91.44 0)
@@
 		(unit 1)
 		(exclude_from_sim no)
-		(in_bom yes)
-		(on_board yes)
-		(dnp no)
+		(in_bom no)
+		(on_board yes)
+		(dnp no)
