File: boards/board-l/board-l.kicad_pcb (KiCad board)
At the start: 2 copper layers, 60 x 60 mm, 74 parts, among them J2 2.54mm 1x6 female, J3 SWD 1x5 (hand-fit), J4 UART pads, SW2 Power ON/OFF slide, U2 AL8860MP-13, U3 STM32G031F8P6, U4 AP63203WU-7

Commit message: update
Other:
- board text added: "rev1"
Changed lines of the file:
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@@
+		(end 43.5 40)
+		(stroke
+			(width 0.05)
+			(type solid)
+		)
+		(fill no)
+		(layer "Dwgs.User")
+	)
+	(gr_rect
+		(start 16.5 0)
 		(end 43.5 40)
 		(stroke
@@
 	)
 	(gr_rect
-		(start 16.5 0)
-		(end 43.5 40)
-		(stroke
-			(width 0.05)
-			(type solid)
-		)
-		(fill no)
-		(layer "Dwgs.User")
-	)
-	(gr_rect
 		(start 0 0)
 		(end 4 4)
@@
 		(layer "User.2")
 	)
+	(gr_text "rev1"
+		(at 58.4 38 90)
+		(layer "B.SilkS")
+		(effects
+			(font
+				(size 1.5 1.5)
+				(thickness 0.3)
+				(bold yes)
+			)
+			(justify left bottom mirror)
+		)
+	)
 	(gr_text "BOARD P REAR ENVELOPE"
