File: boards/swd-adapter/swd-adapter.kicad_pcb (KiCad board)
At the start: 2 copper layers, 36 x 18.1 mm, 2 parts, among them J1 ST-LINK/V2 20-pin (hand-fit), J2 Board L SWD 1x5 (hand-fit)

Commit message: docs: publish SWD adapter evidence and checks
Other:
- board text added: "J2: 1=SWDIO 2=SWCLK 3=NRST 4=VAPP 5=GND"
- board text added: "STRAIGHT PIN-FOR-PIN CABLE"
- board text removed: "1 SWDIO 2 SWCLK 3 NRST 4 VAPP 5 GND"
