File: candidates/board-p-v199-pending-user-decision/board-p-COUT1206-TRIAL.kicad_pcb (KiCad board)
At the start: 2 copper layers, 27 x 40 mm, 27 parts, among them J1 USB4105 TRIAL ADAPTER - UNADO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, U1 HUSB238_006DD - DRAFT LAND / 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, U2 TPS259474LRPWR - TI LAND CAND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

Commit message: feat(candidates): add SMAJ20A input TVS at J1 VBUS to V199
Place DTVS (High Diode SMAJ20A / C571370, retained SMA footprint, pad 1
cathode on RAW_USB_VBUS) left of J1 below MH1. Route it with 0.6 mm F.Cu from
the J1 VBUS via square and a 0.6 mm GND stub to the existing GND track. Add the
schematic symbol, global labels, lib-symbol cache entry, library footprint copy
and BOM row. This is a layout change pending the user's TVS decision.

Co-Authored-By: Claude Opus 5.5 <noreply@anthropic.com>
Claude-Session: https://claude.ai/code/session_01JXThoR3BYUPdQM1u91yCf9
Parts:
- added DTVS: SMAJ20A, zudo-led-lamp:SMA_L4.2-W2.6-LS5.3-RD, F.Cu at (5.60, 10.9)
Routing:
- net RAW_USB_VBUS: track 75.3 -> 84.0 mm
- net GND: track 215.7 -> 218.1 mm
