File: candidates/board-p-rnext-stusb-unadopted/board-p-rnext.kicad_sch (KiCad schematic)
At the start: 54 parts, among them J1 TYPE-C-31-M-17, J2 PogoPad_1x4_NVM_I2C, J3 PogoPad_1x8_Debug, Q1 DMP3036SFG-7, Q3 CSD18543Q3A, Q5 BSS138-7-F, U1 STUSB4500QTR, U2 TPS16630PWPR, U3 LM74700QDBVRQ1, U4 TPS259474LRPWR, U5 TPS3701DDCT

Commit message: r-next candidate: resolve footprints, check lands against manufacturer drawings
Copy 16 zudo-pd footprints unchanged (3ac13d46, hashes recorded) and add
fp-lib-table. Land check vs transcribed TI/Diodes drawings: U2, U4, U5,
Q1, Q3 match; U3, D5, D8 differ, so drafted manufacturer lands are
selected for those; Q5 still differs. Native ERC rerun: footprint-link
warnings 54 -> 0, 13 pin_to_pin remain; netlist PASS. Window check adds
TPS3701 OUTA 300 nA leakage to the U4 UV band.

Co-Authored-By: Claude Opus 5.5 <noreply@anthropic.com>
Claude-Session: https://claude.ai/code/session_01JXThoR3BYUPdQM1u91yCf9
Parts:
- D5: footprint zudo-pd:WSON-6_L2.0-W2.0-P0.65-BL-EP -> rnext-mfr:WSON-6_DRV0006A_TI-EXAMPLE
- D8: footprint zudo-pd:SOD-123_L2.8-W1.8-LS3.7-RD -> rnext-mfr:SOD-123_DIODES-SUGGESTED
- U3: footprint zudo-pd:SOT-23-6_L2.9-W1.6-P0.95-LS2.8-BL -> rnext-mfr:SOT-23-6_DBV0006A_TI-EXAMPLE
Changed lines of the file:
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@@
 			)
 		)
-		(property "Footprint" "zudo-pd:WSON-6_L2.0-W2.0-P0.65-BL-EP"
+		(property "Footprint" "rnext-mfr:WSON-6_DRV0006A_TI-EXAMPLE"
 			(at 203.2 38.1 0)
 			(effects
@@
 			)
 		)
-		(property "Footprint" "zudo-pd:SOT-23-6_L2.9-W1.6-P0.95-LS2.8-BL"
+		(property "Footprint" "rnext-mfr:SOT-23-6_DBV0006A_TI-EXAMPLE"
 			(at 241.3 266.7 0)
 			(effects
@@
 			)
 		)
-		(property "Footprint" "zudo-pd:SOD-123_L2.8-W1.8-LS3.7-RD"
+		(property "Footprint" "rnext-mfr:SOD-123_DIODES-SUGGESTED"
 			(at 279.4 76.2 0)
 			(effects

Commit message: r-next candidate: J3 debug row becomes a 2 x 4 1.5 mm test-pad array
LED per-product population of the common block: same symbol, pins and
nets; courtyard 77.0 -> 18.0 mm2. VBUS_IN sits at a corner next to GND
and VBEN only. J2 (NVM edge-clip row) unchanged, so the jig is unaffected.
Native ERC rerun: 0 errors, 13 pin_to_pin; netlist PASS. Owner bundles
refreshed for the new spec hash, 9/9 PASS.

Co-Authored-By: Claude Opus 5.5 <noreply@anthropic.com>
Claude-Session: https://claude.ai/code/session_01JXThoR3BYUPdQM1u91yCf9
Parts:
- J3: value PogoPad_1x8_Debug -> TestPad_2x4_Debug; footprint zudo-pd:PogoPad_1x08_P2.54mm -> rnext-mfr:TestPadArray_2x4_P1.5_D1.0_J3
Changed lines of the file:
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@@
 			)
 		)
-		(property "Value" "PogoPad_1x8_Debug"
+		(property "Value" "TestPad_2x4_Debug"
 			(at 317.5 195.58 0)
 			(effects
@@
 			)
 		)
-		(property "Footprint" "zudo-pd:PogoPad_1x08_P2.54mm"
+		(property "Footprint" "rnext-mfr:TestPadArray_2x4_P1.5_D1.0_J3"
 			(at 317.5 190.5 0)
 			(effects
